File: KBT1/KBT1.kicad_sch (KiCad schematic)
At the start: 33 parts, among them J1 Conn_01x08_Male, K0 KEYSW, K1 KEYSW, K10 KEYSW, K11 KEYSW, K12 KEYSW, K13 KEYSW, K14 KEYSW, K15 KEYSW, K2 KEYSW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

Commit message: new diode footprint, added mounting holes
Parts:
- added H1, H2, H3, H4: MountingHole, MountingHole:MountingHole_2.7mm, symbol Mechanical:MountingHole
- D1, D10, D12, D13, D14, D15, D16, D2, D3, D4, D5, D6, D7, D8, D9: footprint keyboard_parts:D_SOD123_axial -> Diode_THT:D_DO-35_SOD27_P7.62mm_Horizontal
- D11: footprint Diode_SMD:D_0805_2012Metric_Pad1.15x1.40mm_HandSolder -> Diode_THT:D_DO-35_SOD27_P7.62mm_Horizontal
- J1: footprint Connector_PinHeader_1.00mm:PinHeader_1x08_P1.00mm_Vertical -> Connector_PinHeader_2.54mm:PinHeader_1x08_P2.54mm_Vertical
- K0, K1, K10, K11, K12, K13, K14, K15, K2, K3, K4, K5, K6, K7, K8, K9: footprint Button_Switch_Keyboard:SW_Cherry_MX_1.00u_PCB -> 6:SW_Hotswap_Kailh_MX_plated
