File: Splitboard-A/_autosave-Splitboard-A.kicad_sch (KiCad schematic)
At the start: 111 parts, among them J1 USB_C_Receptacle_USB2.0, J2 USB_C_Receptacle, J3 Conn_01x07, K1 KEYSW, K10 KEYSW, K11 KEYSW, K12 KEYSW, K13 KEYSW, K14 KEYSW, K15 KEYSW, K16 KEYSW, K17 KEYSW, K18 KEYSW, K19 KEYSW, K2 KEYSW, K20 KEYSW, K21 KEYSW, K22 KEYSW, K23 KEYSW, K24 KEYSW, K25 KEYSW, K26 KEYSW, K27 KEYSW, K28 KEYSW, K29 KEYSW, K3 KEYSW, K30 KEYSW, K31 KEYSW, K32 KEYSW, K33 KEYSW, K34 KEYSW, K35 KEYSW, K36 KEYSW, K37 KEYSW, K38 KEYSW, K4 KEYSW, K5 KEYSW, K6 KEYSW, K7 KEYSW, K8 KEYSW, K9 KEYSW, SW1 RotaryEncoder, SW2 SW_Push, U1 AMS1117-3.3, U2 STM32F407VGTx, U3 CR2013-MI2120

Commit message: Schema changes (rotary encoder, debug header)
Parts:
- removed R3, R4: R, symbol Device:R
- added C? (x2): .01uF, symbol Device:C
- added C?: C, symbol Device:C
- added R? (x5): 10k, symbol Device:R
- J3: value Conn_01x07 -> Conn_01x08; symbol Connector_Generic:Conn_01x07 -> Connector_Generic:Conn_01x08
Connections:
- net +3.3V: now also R?.2, R?.2, R?.2
- net ENC_A: now also C?.1, R?.1, R?.1; no longer U2.60 (PD13)
- net ENC_B: now also C?.1, R?.1, R?.1; no longer U2.61 (PD14)
- net GND: now also J3.8 (Pin_8), SW1.S2, C?.1, C?.2, C?.2
- net ENC_SW: now reaches SW1.S1
- net ENC_SW: now also U2.62 (PD15), C?.2, R?.1
- new net ENC_A_F: R?.2, U2.60 (PD13)
- new net ENC_B_F: R?.2, U2.61 (PD14)
Other:
- moved on the sheet: SW1
