File: Splitboard-A/Splitboard-A.kicad_pcb (KiCad board)
At the start: 2 copper layers, 185 x 158.7 mm, 116 parts, among them J1 USB_C_Receptacle_USB2.0, J2 USB_C_Receptacle, J3 Conn_01x07, K1 KEYSW, K10 KEYSW, K11 KEYSW, K12 KEYSW, K13 KEYSW, K14 KEYSW, K15 KEYSW, K16 KEYSW, K17 KEYSW, K18 KEYSW, K19 KEYSW, K2 KEYSW, K20 KEYSW, K21 KEYSW, K22 KEYSW, K23 KEYSW, K24 KEYSW, K25 KEYSW, K26 KEYSW, K27 KEYSW, K28 KEYSW, K29 KEYSW, K3 KEYSW, K30 KEYSW, K31 KEYSW, K32 KEYSW, K33 KEYSW, K34 KEYSW, K35 KEYSW, K36 KEYSW, K37 KEYSW, K38 KEYSW, K4 KEYSW, K5 KEYSW, K6 KEYSW, K7 KEYSW, K8 KEYSW, K9 KEYSW, SW1 RotaryEncoder, SW2 SW_Push, U1 AMS1117-3.3, U2 STM32F407VGTx, U3 CR2013-MI2120

Commit message: keyboard layout changes
Parts:
- moved H4 226.6 mm to (101.0, 44.0)
- moved H2 180.6 mm to (116.0, 122.5)
- moved H3 135.6 mm to (259.5, 46.0)
- moved H1 51.8 mm to (251.5, 161.5)
Routing:
- net +3v3 to micro: track 261.6 -> 291.4 mm, vias 2 -> 3
- net Voltage Regulator Input: track 0.00 -> 17.3 mm, vias 0 -> 1
- net GND: track 203.0 -> 215.6 mm
- added copper zone on B.Cu, net GND
Changed lines of the file:
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@@
   (net 162 "Net-(D40-Pad1)")
   (footprint "MountingHole:MountingHole_2.7mm" (layer "F.Cu")
-    (at 291 167)
+    (at 116 122.5)
     (descr "Mounting Hole 2.7mm, no annular")
     (tags "mounting hole 2.7mm no annular")
@@
     (property "Sheetname" "")
     (attr exclude_from_pos_files)
-    (fp_text reference "H2" (at 0 -3.7) (layer "F.SilkS")
+    (fp_text reference "H2" (at -51.78 -6.28) (layer "F.SilkS")
       (effects (font (size 1 1) (thickness 0.15)))
     )
@@
   )
   (footprint "MountingHole:MountingHole_2.7mm" (layer "F.Cu")
-    (at 303.28 164.08)
+    (at 251.5 161.5)
     (descr "Mounting Hole 2.7mm, no annular")
     (tags "mounting hole 2.7mm no annular")
@@
   )
   (footprint "MountingHole:MountingHole_2.7mm" (layer "F.Cu")
-    (at 298 176)
+    (at 259.5 46)
     (descr "Mounting Hole 2.7mm, no annular")
     (tags "mounting hole 2.7mm no annular")
@@
     (property "Sheetname" "")
     (attr exclude_from_pos_files)
-    (fp_text reference "H3" (at 5.92 -4.7) (layer "F.SilkS")
+    (fp_text reference "H3" (at 4 -0.5) (layer "F.SilkS")
       (effects (font (size 1 1) (thickness 0.15)))
     )
-    (fp_text value "MountingHole" (at 0 3.7) (layer "F.Fab")
+    (fp_text value "MountingHole" (at 1.5 3.7) (layer "F.Fab") hide
       (effects (font (size 1 1) (thickness 0.15)))
     )
@@
   )
   (footprint "MountingHole:MountingHole_2.7mm" (layer "F.Cu")
-    (at 283 179)
+    (at 101 44)
     (descr "Mounting Hole 2.7mm, no annular")
     (tags "mounting hole 2.7mm no annular")
@@
     (property "Sheetname" "")
     (attr exclude_from_pos_files)
-    (fp_text reference "H4" (at 0 -3.7) (layer "F.SilkS")
+    (fp_text reference "H4" (at -2 5) (layer "F.SilkS")
       (effects (font (size 1 1) (thickness 0.15)))
     )
@@
   (segment (start 251.325 81.5) (end 263.190685 81.5) (width 0.25) (layer "B.Cu") (net 25))
   (segment (start 268.05 85.5) (end 269 84.55) (width 0.25) (layer "B.Cu") (net 25))
+  (segment (start 247.591171 59.908829) (end 247.591171 49.53502) (width 0.25) (layer "B.Cu") (net 25))
   (segment (start 266 96) (end 264.959315 96) (width 0.25) (layer "B.Cu") (net 25))
   (segment (start 258.25 145.49) (end 262.5 141.24) (width 0.25) (layer "B.Cu") (net 25))
@@
   (segment (start 269 91.95) (end 269 93.5) (width 0.25) (layer "B.Cu") (net 25))
   (segment (start 266.675 85.5) (end 268.05 85.5) (width 0.25) (layer "B.Cu") (net 25))
+  (segment (start 246 61.5) (end 247.591171 59.908829) (width 0.25) (layer "B.Cu") (net 25))
   (segment (start 265.9 97) (end 265.9 96.1) (width 0.25) (layer "B.Cu") (net 25))
   (segment (start 255.95 156) (end 255.95 149.05) (width 0.25) (layer "B.Cu") (net 25))
@@
   (segment (start 265.75 80.25) (end 265.9125 80.0875) (width 0.25) (layer "F.Cu") (net 54))
   (segment (start 263.5 106.5) (end 268.95 111.95) (width 0.25) (layer "F.Cu") (net 54))
+  (segment (start 234.757352 47.757352) (end 238.5 51.5) (width 0.25) (layer "F.Cu") (net 54))
   (segment (start 265.436396 138.7) (end 262.5 138.7) (width 0.25) (layer "F.Cu") (net 54))
   (segment (start 262.5 80.7755) (end 265.2245 80.7755) (width 0.25) (layer "F.Cu") (net 54))
+  (segment (start 235.21908 43.503397) (end 235.21908 44.310254) (width 0.25) (layer "F.Cu") (net 54))
   (segment (start 263.5 82.5) (end 263.5 106.5) (width 0.25) (layer "F.Cu") (net 54))
+  (segment (start 235.21908 44.310254) (end 234.757352 44.771982) (width 0.25) (layer "F.Cu") (net 54))
+  (segment (start 231.225386 42.049811) (end 231.225386 42.856669) (width 0.25) (layer "F.Cu") (net 54))
+  (segment (start 231.742648 45.242648) (end 234.757352 45.242648) (width 0.25) (layer "F.Cu") (net 54))
   (segment (start 268.95 135.186396) (end 265.436396 138.7) (width 0.25) (layer "F.Cu") (net 54))
+  (segment (start 238.5 51.5) (end 241.5 51.5) (width 0.25) (layer "F.Cu") (net 54))
   (segment (start 265.9125 80.0875) (end 265.9125 78.4125) (width 0.25) (layer "F.Cu") (net 54))
   (segment (start 265.75 80.25) (end 263.5 82.5) (width 0.25) (layer "F.Cu") (net 54))
+  (segment (start 234.757352 45.242648) (end 234.757352 47.757352) (width 0.25) (layer "F.Cu") (net 54))
+  (segment (start 231.225386 42.856669) (end 230.763659 43.318396) (width 0.25) (layer "F.Cu") (net 54))
+  (segment (start 230.763659 43.318396) (end 230.763659 44.263659) (width 0.25) (layer "F.Cu") (net 54))
+  (segment (start 230.763659 44.263659) (end 231.742648 45.242648) (width 0.25) (layer "F.Cu") (net 54))
   (segment (start 268.95 111.95) (end 268.95 135.186396) (width 0.25) (layer "F.Cu") (net 54))
+  (segment (start 234.757352 44.771982) (end 234.757352 45.242648) (width 0.25) (layer "F.Cu") (net 54))
+  (via (at 241.5 51.5) (size 0.8) (drill 0.4) (layers "F.Cu" "B.Cu") (net 54))
   (via (at 262.5 80.7755) (size 0.8) (drill 0.4) (layers "F.Cu" "B.Cu") (net 54))
   (via (at 265.9125 78.4125) (size 0.8) (drill 0.4) (layers "F.Cu" "B.Cu") (net 54))
@@
   (segment (start 251.325 81) (end 262.2755 81) (width 0.25) (layer "B.Cu") (net 54))
   (segment (start 250.5 81) (end 249 79.5) (width 0.25) (layer "B.Cu") (net 54))
+  (segment (start 241.5 60.95) (end 242.05 61.5) (width 0.25) (layer "B.Cu") (net 54))
+  (segment (start 241.5 51.5) (end 241.5 60.95) (width 0.25) (layer "B.Cu") (net 54))
   (segment (start 265.9125 78.4125) (end 265 79.325) (width 0.25) (layer "B.Cu") (net 54))
   (segment (start 245 119) (end 243 119) (width 0.25) (layer "B.Cu") (net 54))
@@
   (segment (start 250.5875 137.5) (end 250.5875 134.5) (width 0.25) (layer "B.Cu") (net 79))
   (segment (start 234.45 137.5) (end 250.5875 137.5) (width 0.25) (layer "B.Cu") (net 79))
+  (segment (start 247.729878 47.5) (end 252.5 47.5) (width 0.25) (layer "F.Cu") (net 91))
+  (segment (start 243.782598 46) (end 247 46) (width 0.25) (layer "F.Cu") (net 91))
+  (segment (start 243.260466 46.522132) (end 243.260466 47.32899) (width 0.25) (layer "F.Cu") (net 91))
+  (segment (start 247.25416 47.975718) (end 247.25416 48.782575) (width 0.25) (layer "F.Cu") (net 91))
+  (segment (start 243.260466 46.522132) (end 243.782598 46) (width 0.25) (layer "F.Cu") (net 91))
+  (segment (start 247 46) (end 247.729878 46.729878) (width 0.25) (layer "F.Cu") (net 91))
+  (segment (start 243.260466 47.32899) (end 242.798739 47.790717) (width 0.25) (layer "F.Cu") (net 91))
+  (segment (start 247.729878 46.729878) (end 247.729878 47.5) (width 0.25) (layer "F.Cu") (net 91))
+  (segment (start 247.25416 47.975718) (end 247.729878 47.5) (width 0.25) (layer "F.Cu") (net 91))
+  (segment (start 247.25416 48.782575) (end 246.792432 49.244303) (width 0.25) (layer "F.Cu") (net 91))
+  (via (at 252.5 47.5) (size 0.8) (drill 0.4) (layers "F.Cu" "B.Cu") (net 91))
+  (segment (start 255.5 47.85) (end 252.85 47.85) (width 0.25) (layer "B.Cu") (net 91))
+  (segment (start 252.85 47.85) (end 252.5 47.5) (width 0.25) (layer "B.Cu") (net 91))
   (segment (start 264.6 63.2) (end 260.8875 63.2) (width 0.25) (layer "B.Cu") (net 92))
   (segment (start 260.8875 63.2) (end 260.5 63.5875) (width 0.25) (layer "B.Cu") (net 92))
@@
   (segment (start 264.65 51.15) (end 266.5 53) (width 0.25) (layer "B.Cu") (net 162))
   (segment (start 255.5 51.15) (end 264.65 51.15) (width 0.25) (layer "B.Cu") (net 162))
+  (zone (net 25) (net_name "GND") (layer "B.Cu") (hatch edge 0.508)
+    (connect_pads yes (clearance 0.2))
+    (min_thickness 0.254) (filled_areas_thickness no)
+    (fill yes (thermal_gap 0.508) (thermal_bridge_width 0.508) (smoothing fillet) (radius 1))
+    (polygon
+      (pts
+        (xy 253.5 41.5)
+        (xy 250 52)
+        (xy 226.5 43.5)
+        (xy 230.5 33)
+      )
+    )
+  )
 )

Commit message: layout updates
Connections:
- C10 pad 1: +3v3 to micro -> VDD
- C11 pad 1: +3v3 to micro -> VDD
- C12 pad 1: +3v3 to micro -> VDD
- C13 pad 1: +3v3 to micro -> VDD
- C14 pad 1: +3v3 to micro -> VDD
- C15 pad 1: +3v3 to micro -> VDD
- C16 pad 1: +3v3 to micro -> VDD
- C17 pad 1: +3v3 to micro -> VDD
- C8 pad 1: +3v3 to micro -> VDD
- C9 pad 1: +3v3 to micro -> VDD
- D41 pad 1: +3v3 to micro -> VDD
- J2 pad A4: +3v3 to micro -> VDD
- J2 pad A9: +3v3 to micro -> VDD
- J2 pad B4: +3v3 to micro -> VDD
- J2 pad B9: +3v3 to micro -> VDD
- J3 pad 6: +3v3 to micro -> VDD
- R1 pad 1: +3v3 to micro -> VDD
- R1 pad 2: +3v3 to micro -> VDD
- R2 pad 2: +3v3 to micro -> VDD
- R3 pad 1: +3v3 to micro -> VDD
- R6 pad 1: +3v3 to micro -> VDD
- U2 pad 100: +3v3 to micro -> VDD
- U2 pad 11: +3v3 to micro -> VDD
- U2 pad 19: +3v3 to micro -> VDD
- U2 pad 28: +3v3 to micro -> VDD
- U2 pad 50: +3v3 to micro -> VDD
- U2 pad 75: +3v3 to micro -> VDD
- U3 pad 1: +3v3 to micro -> VDD
Routing:
- net VDD: track 0.00 -> 291.4 mm, vias 0 -> 3
- net +3v3 to micro: track 291.4 -> 0.00 mm, vias 3 -> 0

Commit message: Added Joe's suggestions & notes to schematic & pcb
Other:
- board text added: "ALL VIA INTERAL DIAMETERS NEED TO BE >= 5mm (for fly wiring) Also untented"
- board text added: "Once done routing, for unused pins, draw out traces and attach vias (assign nets in schematic) this will allow fly wiring if we smoke a pin"
- board text added: "USB receptacles should be spaced a little farther apart to account for usb cable housing clearance (cables may hit each other)"
Changed lines of the file:
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@@
   (gr_line (start 184 126) (end 94 126) (layer "Edge.Cuts") (width 0.1))
   (gr_line (start 94 126) (end 94 31) (layer "Edge.Cuts") (width 0.1))
+  (gr_text "Once done routing, for unused pins,\ndraw out traces and attach vias (assign nets in schematic)\nthis will allow fly wiring if we smoke a pin" (at 317.5 53.34) (layer "F.SilkS")
+    (effects (font (size 1.5 1.5) (thickness 0.3)))
+  )
+  (gr_text "ALL VIA INTERAL DIAMETERS\nNEED TO BE >= 5mm (for fly wiring)\nAlso untented" (at 317.5 68.58) (layer "F.SilkS")
+    (effects (font (size 2 2) (thickness 0.3)))
+  )
+  (gr_text "USB receptacles should be spaced a little farther apart\nto account for usb cable housing clearance\n(cables may hit each other)" (at 251.46 17.78) (layer "F.SilkS")
+    (effects (font (size 1.5 1.5) (thickness 0.3)))
+  )
   (segment (start 229.5875 132.5) (end 229.5875 134.9875) (width 0.25) (layer "B.Cu") (net 1))
   (segment (start 229.5875 134.9875) (end 229.6 135) (width 0.25) (layer "B.Cu") (net 1))

Commit message: updated USB, LCD, ESD, Voltage Reg in schematic
Other:
- board text added: "Mounting holes are cutting into traces, we need to consider creating more board for these holes also consider the screw head that will rest on top of the hole"
- board text added: "The switches unfortunately need to be re-spaced. They are 19mm apart from center to center, we need the horizontal distance to be 19mm, center to center distance will likely be greater than 19mm"
Changed lines of the file:
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@@
+    (effects (font (size 1.5 1.5) (thickness 0.3)))
+  )
+  (gr_text "The switches unfortunately need to be re-spaced.\nThey are 19mm apart from center to center, we need\nthe horizontal distance to be 19mm, center to center\ndistance will likely be greater than 19mm" (at 88.9 17.78) (layer "F.SilkS")
     (effects (font (size 1.5 1.5) (thickness 0.3)))
   )
@@
     (effects (font (size 1.5 1.5) (thickness 0.3)))
   )
+  (gr_text "Mounting holes are cutting into traces,\nwe need to consider creating more board for these holes\nalso consider the screw head that will rest on top of the hole" (at 109.22 139.7) (layer "F.SilkS")
+    (effects (font (size 1.5 1.5) (thickness 0.3)))
+  )

Commit message: Added debugging header to splitboard B
Other:
- board text added: "The switches unfortunately need to be re-spaced. They are 19mm apart from center to center, we need the horizontal distance to be 19mm, center to center distance will be greater than 19mm because of trig & stuff"
- board text removed: "The switches unfortunately need to be re-spaced. They are 19mm apart from center to center, we need the horizontal distance to be 19mm, center to center distance will likely be greater than 19mm"
Changed lines of the file:
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@@
     (effects (font (size 1.5 1.5) (thickness 0.3)))
   )
-  (gr_text "The switches unfortunately need to be re-spaced.\nThey are 19mm apart from center to center, we need\nthe horizontal distance to be 19mm, center to center\ndistance will likely be greater than 19mm" (at 88.9 17.78) (layer "F.SilkS")
+  (gr_text "The switches unfortunately need to be re-spaced.\nThey are 19mm apart from center to center, we need\nthe horizontal distance to be 19mm, center to center\ndistance will be greater than 19mm because of trig & stuff" (at 88.9 17.78) (layer "F.SilkS")
     (effects (font (size 1.5 1.5) (thickness 0.3)))
   )
