File: Splitboard-A/Splitboard-A.kicad_pcb (KiCad board)
At the start: 2 copper layers, 185 x 158.7 mm, 116 parts, among them J1 USB_C_Receptacle_USB2.0, J2 USB_C_Receptacle, J3 Conn_01x07, K1 KEYSW, K10 KEYSW, K11 KEYSW, K12 KEYSW, K13 KEYSW, K14 KEYSW, K15 KEYSW, K16 KEYSW, K17 KEYSW, K18 KEYSW, K19 KEYSW, K2 KEYSW, K20 KEYSW, K21 KEYSW, K22 KEYSW, K23 KEYSW, K24 KEYSW, K25 KEYSW, K26 KEYSW, K27 KEYSW, K28 KEYSW, K29 KEYSW, K3 KEYSW, K30 KEYSW, K31 KEYSW, K32 KEYSW, K33 KEYSW, K34 KEYSW, K35 KEYSW, K36 KEYSW, K37 KEYSW, K38 KEYSW, K4 KEYSW, K5 KEYSW, K6 KEYSW, K7 KEYSW, K8 KEYSW, K9 KEYSW, SW1 RotaryEncoder, SW2 SW_Push, U1 AMS1117-3.3, U2 STM32F407VGTx, U3 CR2013-MI2120

Commit message: Layout changes
Parts:
- removed D40, D41, D42: D_Schottky, Diode_SMD:D_SOD-123
- removed F1: 500mA, Fuse:Fuse_BelFuse_0ZRE0125FF_L21.2mm_W5.3mm
- added C18: 100nF, Capacitor_SMD:C_0805_2012Metric, B.Cu at (247.9, 116.5)
- added D39: D_Schottky, Diode_SMD:D_SOD-123, B.Cu at (264.5, 45.0)
- added R10: 10k, Resistor_SMD:R_0805_2012Metric, B.Cu at (252.0, 139.0)
- added R11: 10k, Resistor_SMD:R_0805_2012Metric, B.Cu at (230.5, 132.5)
- added R12: 10k, Resistor_SMD:R_0805_2012Metric, B.Cu at (230.5, 129.4)
- added R13: 10k, Resistor_SMD:R_0805_2012Metric, B.Cu at (230.5, 137.5)
- added R14: 10k, Resistor_SMD:R_0805_2012Metric, B.Cu at (226.5, 133.4)
- added R15: 10K, Resistor_SMD:R_0805_2012Metric, B.Cu at (271.5, 87.5)
- added R7: 10k, Resistor_SMD:R_0805_2012Metric, B.Cu at (237.5, 82.0)
- added R8: 10k, Resistor_SMD:R_0805_2012Metric, B.Cu at (237.5, 79.5)
- added R9: 10k, Resistor_SMD:R_0805_2012Metric, B.Cu at (237.5, 77.0)
- added U4: AMS1117-3.3, Package_TO_SOT_SMD:SOT-223-3_TabPin2, B.Cu at (264.5, 52.0)
- added U5: USBUF02W6, ul_USBUF02W6:USBUF02W6, B.Cu at (250.5, 55.5)
- C1: value 0.1uF -> 2u2; footprint Resistor_SMD:R_0805_2012Metric -> Capacitor_SMD:C_0805_2012Metric
- C16, C17: value 100nF -> .01uF
- C2: value 10u -> 2u2
- C4: value .01uF -> 10u
- C5: value .01uF -> 100nF
- C6: value 100nF -> 10uf
- C8: value 1uf -> 100nF
- H1, H2, H3, H4: moved to B.Cu
- J2: footprint Connector_USB:USB_C_Receptacle_GCT_USB4085 -> Connector_USB:USB_C_Receptacle_Amphenol_12401548E4-2A
- J3: value Conn_01x07 -> Conn_01x06; footprint Connector_PinHeader_2.54mm:PinHeader_1x07_P2.54mm_Horizontal -> Connector_PinHeader_2.54mm:PinHeader_1x06_P2.54mm_Horizontal
- R1: value 10K -> 5K1
- R2: value 100K -> 5K1
- SW1: footprint Rotary_Encoder:RotaryEncoder_Alps_EC12E_Vertical_H20mm -> Rotary_Encoder:RotaryEncoder_Alps_EC11E-Switch_Vertical_H20mm
- SW2: footprint Button_Switch_SMD:Nidec_Copal_SH-7010A -> Button_Switch_THT:SW_PUSH_6mm
- U1: value AMS1117-3.3 -> SIT2024BA-S2-33E-8.000000G; footprint Package_TO_SOT_SMD:SOT-223-3_TabPin2 -> SIT2024BA:SIT2024BA-S2-33E-8.000000G
- U2: value STM32F407VGTx -> CR2013-MI2120; footprint Package_QFP:LQFP-100_14x14mm_P0.5mm -> Display:CR2013-MI2120
- U3: value CR2013-MI2120 -> STM32F407VGTx; footprint Display:CR2013-MI2120 -> Package_QFP:LQFP-100_14x14mm_P0.5mm; moved to B.Cu
- moved H1 111.6 mm to (273.0, 52.0), turned to 180 degrees
- moved H3 109.2 mm to (253.0, 155.0), turned to 180 degrees
- moved H2 94.1 mm to (112.5, 28.5), turned to 180 degrees
- moved H4 80.6 mm to (117.0, 123.0), turned to 180 degrees
- moved C7 59.1 mm to (251.0, 97.0), turned to -90 degrees
- moved R6 54.8 mm to (237.5, 84.5), turned to 0 degrees
- moved R5 50.6 mm to (241.0, 85.0), turned to 90 degrees
- moved R4 49.3 mm to (243.5, 84.9), turned to 90 degrees
- moved C16 46.9 mm to (228.5, 126.5), turned to 180 degrees
- moved SW2 42.8 mm to (247.0, 108.5)
- moved C17 42.1 mm to (225.0, 130.0), turned to 0 degrees
- moved U2 37.3 mm to (263.7, 124.0), turned to 90 degrees
- moved U3 34.9 mm to (259.0, 87.0), turned to 180 degrees
- moved C1 31.5 mm to (254.5, 97.0), turned to 0 degrees
- moved U1 31.5 mm to (270.9, 81.2)
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Connections:
- C1 pad 1: +3v3 to micro -> Net-(C1-Pad1)
- C10 pad 1: VDD -> +3.3V
- C11 pad 1: VDD -> +3.3V
- C12 pad 1: VDD -> +3.3V
- C13 pad 1: VDD -> +3.3V
- C14 pad 1: VDD -> +3.3V
- C15 pad 1: VDD -> +3.3V
- C16 pad 1: VDD -> /ENC_A
- C17 pad 1: VDD -> GND
- C17 pad 2: GND -> /ENC_B
- C3 pad 1: +3v3 to micro -> Net-(C3-Pad1)
- C4 pad 1: /ENC_A -> +3.3V
- C5 pad 2: /ENC_B -> /ENC_SW
- C6 pad 1: GND -> +3.3V
- C6 pad 2: /ENC_SW -> GND
- C7 pad 1: GND -> +3.3V
- C7 pad 2: /NRST -> GND
- C8 pad 1: VDD -> +3.3V
- C9 pad 1: VDD -> +3.3V
- FB1 pad 2: Net-(C2-Pad1) -> Net-(C3-Pad1)
- J1 pad A4: Voltage Regulator Input -> VBUS
- J1 pad A5: unconnected-(J1-PadA5) -> Net-(J1-PadA5)
- J1 pad A6: /USB_DP -> /USB_CONN_D+
- J1 pad A7: /USB_DM -> /USB_CONN_D-
- J1 pad A9: Voltage Regulator Input -> VBUS
- J1 pad B4: Voltage Regulator Input -> VBUS
- J1 pad B5: unconnected-(J1-PadB5) -> Net-(J1-PadB5)
- J1 pad B6: unconnected-(J1-PadB6) -> /USB_CONN_D+
- J1 pad B7: unconnected-(J1-PadB7) -> /USB_CONN_D-
- J1 pad B9: Voltage Regulator Input -> VBUS
- J2 pad A4: VDD -> VBUS
- J2 pad A5: unconnected-(J2-PadA5) -> /MOSI
- J2 pad A6: unconnected-(J2-PadA6) -> /SDA
- J2 pad A7: unconnected-(J2-PadA7) -> /SCL
- J2 pad A8: unconnected-(J2-PadA8) -> /SCK
- J2 pad A9: VDD -> VBUS
- J2 pad B4: VDD -> VBUS
- J2 pad B5: unconnected-(J2-PadB5) -> /MOSI
- J2 pad B6: unconnected-(J2-PadB6) -> /SDA
- J2 pad B7: unconnected-(J2-PadB7) -> /SCL
- J2 pad B8: unconnected-(J2-PadB8) -> /SCK
- J2 pad B9: VDD -> VBUS
- J3 pad 1: GND -> +3.3V
- J3 pad 2: /SWDIO -> /SWCLK
- J3 pad 3: /SWCLK -> GND
- J3 pad 4: /TRST -> /SWDIO
- J3 pad 5: /SWO -> /NRST
- J3 pad 6: VDD -> /SWO
- R1 pad 1: VDD -> Net-(J1-PadA5)
- R1 pad 2: VDD -> GND
- R2 pad 1: +3v3 to micro -> Net-(J1-PadB5)
- R2 pad 2: VDD -> GND
- R3 pad 1: VDD -> /ENC_SW
- R3 pad 2: Net-(R3-Pad2) -> +3.3V
- R4 pad 1: /ENC_A -> /col5
- R4 pad 2: Net-(R3-Pad2) -> +3.3V
- R5 pad 1: Net-(R5-Pad1) -> /col4
- R5 pad 2: /ENC_B -> +3.3V
- R6 pad 1: VDD -> /col3
- R6 pad 2: Net-(R5-Pad1) -> +3.3V
- SW1 pad A: Net-(R3-Pad2) -> Net-(R11-Pad2)
- SW1 pad B: Net-(R5-Pad1) -> Net-(R13-Pad2)
- U1 pad 2: +3v3 to micro -> unconnected-(U1-Pad2)
- U1 pad 3: Net-(C2-Pad1) -> unconnected-(U1-Pad3)
- U2 pad 1: unconnected-(U2-Pad1) -> VBUS
- U2 pad 10: GND -> unconnected-(U2-Pad10)
- U2 pad 11: VDD -> unconnected-(U2-Pad11)
- U2 pad 14: /NRST -> unconnected-(U2-Pad14)
- U2 pad 2: unconnected-(U2-Pad2) -> GND
- U2 pad 3: unconnected-(U2-Pad3) -> /LCD1_CS
- U2 pad 4: unconnected-(U2-Pad4) -> /LCD1_RST
- U2 pad 5: unconnected-(U2-Pad5) -> /LCD1_DC
- U2 pad 6: unconnected-(U2-Pad6) -> /MOSI
- U2 pad 7: unconnected-(U2-Pad7) -> /SCK
- U2 pad 8: unconnected-(U2-Pad8) -> +3.3V
- U3 pad 1: VDD -> unconnected-(U3-Pad1)
- U3 pad 10: unconnected-(U3-Pad10) -> GND
- U3 pad 11: unconnected-(U3-Pad11) -> +3.3V
- U3 pad 12: unconnected-(U3-Pad12) -> /RCC_OSC_IN
- U3 pad 13: unconnected-(U3-Pad13) -> /RCC_OSC_OUT
- U3 pad 14: unconnected-(U3-Pad14) -> /NRST
- U3 pad 2: GND -> unconnected-(U3-Pad2)
- U3 pad 3: /CS -> unconnected-(U3-Pad3)
- U3 pad 6: /MOSI -> +3.3V
- U3 pad 7: /SCK -> unconnected-(U3-Pad7)
- U3 pad 9: /MISO -> unconnected-(U3-Pad9)
Routing:
- net VDD: track 291.4 -> 0.00 mm, vias 3 -> 0
- net +3.3V: track 0.00 -> 232.6 mm, vias 0 -> 7
- net /MOSI: track 0.00 -> 169.9 mm, vias 0 -> 2
- net VBUS: track 0.00 -> 149.5 mm, vias 0 -> 4
- net /SCK: track 0.00 -> 104.6 mm, vias 0 -> 1
- net /ENC_B: track 2.51 -> 70.0 mm, vias 0 -> 2
- net /ENC_SW: track 0.00 -> 66.7 mm, vias 0 -> 1
- net /LCD2_DC: track 0.00 -> 66.2 mm, vias 0 -> 1
- net GND: track 215.6 -> 277.7 mm, vias 0 -> 4
- net /SCL: track 0.00 -> 61.2 mm, vias 0 -> 1
- net /TRST: track 60.8 -> 0.00 mm, vias 1 -> 0
- net /SDA: track 0.00 -> 60.2 mm, vias 0 -> 1
- net /LCD2_CS: track 0.00 -> 56.9 mm, vias 0 -> 1
- net /ENC_A: track 2.51 -> 52.3 mm, vias 0 -> 2
- net /LCD2_RST: track 0.00 -> 48.8 mm, vias 0 -> 1
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- added copper zone on B.Cu, net +3.3V
Other:
- board size 185 x 158.7 mm -> 185 x 161.7 mm

Commit message: added more archive files
Parts:
- U1: value SIT2024BA-S2-33E-8.000000G -> SIT2024BA
Changed lines of the file:
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@@
       (effects (font (size 1 1) (thickness 0.15)) (justify mirror))
     )
-    (fp_text value "SIT2024BA-S2-33E-8.000000G" (at 0 0) (layer "B.SilkS")
+    (fp_text value "SIT2024BA" (at -3.4465 -0.0815 90) (layer "B.SilkS")
       (effects (font (size 1 1) (thickness 0.15)) (justify mirror))
     )
@@
       (effects (font (size 1 1) (thickness 0.15)) (justify mirror))
     )
-    (fp_text value "100nF" (at 50.18 46.39 90) (layer "B.Fab")
+    (fp_text value "100nF" (at 1.68 2.78 90) (layer "B.Fab")
       (effects (font (size 1 1) (thickness 0.15)) (justify mirror))
     )
@@
   (gr_line (start 279 127) (end 279 142) (layer "Edge.Cuts") (width 0.1))
   (gr_arc (start 94 28.5) (mid 188.364195 21.256196) (end 279 48.5) (layer "Edge.Cuts") (width 0.1))
-  (gr_text "Once done routing, for unused pins,\ndraw out traces and attach vias (assign nets in schematic)\nthis will allow fly wiring if we smoke a pin" (at 341 54) (layer "F.SilkS")
+  (gr_text "Once done routing, for unused pins,\ndraw out traces and attach vias (assign nets in schematic)\nthis will allow fly wiring if we smoke a pin" (at 368.3 88.9) (layer "F.SilkS")
     (effects (font (size 1.5 1.5) (thickness 0.3)))
   )
-  (gr_text "The switches unfortunately need to be re-spaced.\nThey are 19mm apart from center to center, we need\nthe horizontal distance to be 19mm, center to center\ndistance will be greater than 19mm because of trig & stuff" (at 88.9 17.78) (layer "F.SilkS")
+  (gr_text "The switches unfortunately need to be re-spaced.\nThey are 19mm apart from center to center, we need\nthe horizontal distance to be 19mm, center to center\ndistance will be greater than 19mm because of trig & stuff" (at 48.26 -7.62) (layer "F.SilkS")
     (effects (font (size 1.5 1.5) (thickness 0.3)))
   )
-  (gr_text "ALL VIA INTERAL DIAMETERS\nNEED TO BE >= 5mm (for fly wiring)\nAlso untented" (at 335.5 73.5) (layer "F.SilkS")
+  (gr_text "ALL VIA INTERAL DIAMETERS\nNEED TO BE >= 5mm (for fly wiring)\nAlso untented" (at 373.38 109.22) (layer "F.SilkS")
     (effects (font (size 2 2) (thickness 0.3)))
   )
-  (gr_text "USB receptacles should be spaced a little farther apart\nto account for usb cable housing clearance\n(cables may hit each other)" (at 251.46 17.78) (layer "F.SilkS")
+  (gr_text "USB receptacles should be spaced a little farther apart\nto account for usb cable housing clearance\n(cables may hit each other)" (at 373.38 22.86) (layer "F.SilkS")
     (effects (font (size 1.5 1.5) (thickness 0.3)))
   )
-  (gr_text "Mounting holes are cutting into traces,\nwe need to consider creating more board for these holes\nalso consider the screw head that will rest on top of the hole" (at 109.22 139.7) (layer "F.SilkS")
+  (gr_text "Mounting holes are cutting into traces,\nwe need to consider creating more board for these holes\nalso consider the screw head that will rest on top of the hole" (at 53.34 208.28) (layer "F.SilkS")
     (effects (font (size 1.5 1.5) (thickness 0.3)))
   )

Commit message: Layout changes
Parts:
- added C19: 10uf, Capacitor_SMD:C_0805_2012Metric, B.Cu at (261.9, 46.9)
- added C20: 100nF, Capacitor_SMD:C_0805_2012Metric, B.Cu at (265.3, 46.9)
- added C21: 100nF, Capacitor_SMD:C_0805_2012Metric, B.Cu at (274.5, 81.2)
- added D40: D_Schottky, Diode_SMD:D_SOD-123, B.Cu at (229.5, 52.5)
- added D41: D_Schottky, Diode_SMD:D_SOD-123, B.Cu at (261.0, 100.5)
- added R16: 20, Resistor_SMD:R_0805_2012Metric, B.Cu at (259.1, 63.8)
- added R17: 20, Resistor_SMD:R_0805_2012Metric, B.Cu at (256.8, 63.8)
- added R18: 20, Resistor_SMD:R_0805_2012Metric, B.Cu at (263.7, 63.8)
- added R19: 20, Resistor_SMD:R_0805_2012Metric, B.Cu at (261.4, 63.8)
- added R20: 20, Resistor_SMD:R_0805_2012Metric, B.Cu at (265.9, 63.8)
- added R21: 20, Resistor_SMD:R_0805_2012Metric, B.Cu at (252.1, 63.8)
- added R22: 20, Resistor_SMD:R_0805_2012Metric, B.Cu at (234.3, 141.1)
- added R23: 20, Resistor_SMD:R_0805_2012Metric, B.Cu at (247.5, 73.5)
- added R24: 20, Resistor_SMD:R_0805_2012Metric, B.Cu at (249.6, 73.5)
- added R25: 20, Resistor_SMD:R_0805_2012Metric, B.Cu at (251.7, 73.5)
- added R26: 20, Resistor_SMD:R_0805_2012Metric, B.Cu at (253.8, 73.5)
- added R27: 20, Resistor_SMD:R_0805_2012Metric, B.Cu at (255.9, 73.5)
- added R28: 20, Resistor_SMD:R_0805_2012Metric, B.Cu at (258.0, 73.5)
- added R29: 20, Resistor_SMD:R_0805_2012Metric, B.Cu at (260.1, 73.5)
- added R30: 20, Resistor_SMD:R_0805_2012Metric, B.Cu at (262.2, 73.5)
- added R31: 20, Resistor_SMD:R_0805_2012Metric, B.Cu at (246.9, 98.2)
- added R32: 20, Resistor_SMD:R_0805_2012Metric, B.Cu at (246.9, 95.8)
- added R33: 20, Resistor_SMD:R_0805_2012Metric, B.Cu at (246.9, 93.5)
- added R34: 20, Resistor_SMD:R_0805_2012Metric, B.Cu at (246.9, 91.2)
- added R35: 20, Resistor_SMD:R_0805_2012Metric, B.Cu at (246.9, 89.0)
- added R36: 20, Resistor_SMD:R_0805_2012Metric, B.Cu at (241.1, 129.7)
- added R37: 20, Resistor_SMD:R_0805_2012Metric, B.Cu at (263.4, 142.5)
- added R38: 4k7, Resistor_SMD:R_0805_2012Metric, B.Cu at (271.9, 70.6)
- added R39: 4k7, Resistor_SMD:R_0805_2012Metric, B.Cu at (271.9, 68.3)
- J1: footprint Connector_USB:USB_C_Receptacle_GCT_USB4085 -> Connector_USB:USB_C_Receptacle_Amphenol_12401548E4-2A
- R3: value 10k -> 20
- U1: value SIT2024BA -> SIT2024BA-S2-33E-8.000000G
- moved C4 77.9 mm to (229.4, 57.1), turned to -90 degrees
- moved R3 75.1 mm to (254.4, 63.8), turned to 90 degrees
- moved U4 27.8 mm to (236.7, 53.5), turned to 180 degrees
- moved R2 27.1 mm to (231.1, 46.3)
- moved C8 26.3 mm to (264.0, 97.0), turned to 0 degrees
- moved C17 23.9 mm to (241.1, 147.7), turned to 180 degrees
- moved D39 21.3 mm to (244.0, 50.8), turned to 90 degrees
- moved R1 19.1 mm to (228.9, 46.3), turned to -90 degrees
- moved R14 18.7 mm to (241.1, 145.1), turned to 180 degrees
- moved FB1 18.7 mm to (244.2, 54.4), turned to 180 degrees
- moved U5 18.5 mm to (234.2, 46.7), turned to 0 degrees
- moved J2 16.7 mm to (252.2, 44.2)
- moved J1 15.5 mm to (236.2, 38.5)
- moved C16 13.9 mm to (241.1, 132.3), turned to 0 degrees
- moved C3 13.3 mm to (244.2, 56.8), turned to 0 degrees
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Connections:
- C4 pad 1: +3.3V -> Net-(C4-Pad1)
- J2 pad A10: /LCD2_CS -> Net-(J2-PadA10)
- J2 pad A11: /LCD2_DC -> Net-(J2-PadA11)
- J2 pad A2: unconnected-(J2-PadA2) -> Net-(J2-PadA2)
- J2 pad A3: /LCD2_RST -> Net-(J2-PadA3)
- J2 pad A5: /MOSI -> Net-(J2-PadA5)
- J2 pad A6: /SDA -> Net-(J2-PadA6)
- J2 pad A7: /SCL -> Net-(J2-PadA7)
- J2 pad A8: /SCK -> Net-(J2-PadA8)
- J2 pad B10: /LCD2_CS -> Net-(J2-PadA10)
- J2 pad B11: /LCD2_DC -> Net-(J2-PadA11)
- J2 pad B2: unconnected-(J2-PadB2) -> Net-(J2-PadA2)
- J2 pad B3: /LCD2_RST -> Net-(J2-PadA3)
- J2 pad B5: /MOSI -> Net-(J2-PadA5)
- J2 pad B6: /SDA -> Net-(J2-PadA6)
- J2 pad B7: /SCL -> Net-(J2-PadA7)
- J2 pad B8: /SCK -> Net-(J2-PadA8)
- J3 pad 1: +3.3V -> Net-(J3-Pad1)
- R3 pad 1: /ENC_SW -> /MOSI
- R3 pad 2: +3.3V -> Net-(J2-PadA5)
- U1 pad 3: unconnected-(U1-Pad3) -> +3.3V
- U3 pad 55: /col1 -> Net-(U3-Pad55)
- U3 pad 56: /col2 -> Net-(U3-Pad56)
- U3 pad 57: /col3 -> Net-(U3-Pad57)
- U3 pad 58: /col4 -> Net-(U3-Pad58)
- U3 pad 59: /col5 -> Net-(U3-Pad59)
- U3 pad 60: /ENC_A -> Net-(U3-Pad60)
- U3 pad 61: /ENC_B -> Net-(U3-Pad61)
- U3 pad 62: /ENC_SW -> Net-(U3-Pad62)
- U3 pad 81: /row0 -> Net-(U3-Pad81)
- U3 pad 82: /row1 -> Net-(U3-Pad82)
- U3 pad 83: /row2 -> Net-(U3-Pad83)
- U3 pad 84: /row3 -> Net-(U3-Pad84)
- U3 pad 85: /row4 -> Net-(U3-Pad85)
- U3 pad 86: /row5 -> Net-(U3-Pad86)
- U3 pad 87: /row6 -> Net-(U3-Pad87)
- U3 pad 88: /col0 -> Net-(U3-Pad88)
- U4 pad 2: +3.3V -> Net-(C4-Pad1)
Routing:
- net /MOSI: track 169.9 -> 87.2 mm
- net Net-(U3-Pad62): track 0.00 -> 80.1 mm, vias 0 -> 2
- net Net-(U3-Pad61): track 0.00 -> 64.5 mm, vias 0 -> 2
- net /ENC_B: track 70.0 -> 9.73 mm, vias 2 -> 0
- net /row0: track 276.3 -> 335.0 mm
- net /ENC_SW: track 66.7 -> 9.27 mm, vias 1 -> 0
- net Net-(J2-PadA7): track 0.00 -> 57.3 mm, vias 0 -> 2
- net Net-(U3-Pad60): track 0.00 -> 53.5 mm, vias 0 -> 2
- net Net-(J2-PadA5): track 0.00 -> 50.2 mm, vias 0 -> 1
- net /ENC_A: track 52.3 -> 5.18 mm, vias 2 -> 0
- net Net-(J2-PadA8): track 0.00 -> 43.0 mm, vias 0 -> 2
- net Net-(J2-PadA10): track 0.00 -> 40.9 mm, vias 0 -> 1
- net Net-(J2-PadA3): track 0.00 -> 40.5 mm, vias 0 -> 2
- net Net-(J2-PadA11): track 0.00 -> 37.9 mm, vias 0 -> 3
- net Net-(D39-Pad1): track 33.7 -> 2.41 mm
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Other:
- outline, holes or cut-outs redrawn
- board text added: "1"
- board text added: "Split Keyboard Side A ECE 477 Group 4 Fall 2022 Senior Design Andrew Smolensky Logan Stapleton Joe Zobel Justin Selbo"

Commit message: Layout changes
Parts:
- J3: moved to B.Cu
- U2: moved to F.Cu
- moved U2 20.3 mm to (243.4, 123.8)
- moved SW2 6.50 mm to (240.5, 108.5)
- turned J3 to 180 degrees
Routing:
- net +3.3V: track 251.8 -> 228.5 mm, vias 9 -> 8
- net VBUS: track 133.2 -> 153.8 mm
- net GND: track 303.8 -> 314.6 mm
- net /SCK: track 96.3 -> 86.8 mm, vias 3 -> 2
- net /MOSI: track 87.2 -> 78.6 mm
- net /LCD1_RST: track 51.0 -> 58.3 mm
- net /NRST: track 60.8 -> 67.3 mm, vias 3 -> 4
- net Net-(U3-Pad61): track 64.5 -> 68.8 mm
- net /LCD1_DC: track 48.1 -> 50.9 mm
- net /LCD1_CS: track 48.9 -> 46.2 mm
- net /row5: track 143.2 -> 140.8 mm
- net /row4: track 159.6 -> 157.5 mm
- net /row6: track 123.5 -> 121.9 mm
- net Net-(U3-Pad60): track 53.5 -> 52.1 mm
- net Net-(U3-Pad62): track 80.1 -> 79.1 mm
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Other:
- board text added: "TO PC"
- board text added: "TO SIDE B"

Commit message: Addes rseries for LCD and added extra vias
Parts:
- added R40: 20, Resistor_SMD:R_0805_2012Metric, B.Cu at (243.3, 115.9)
- added R41: 20, Resistor_SMD:R_0805_2012Metric, B.Cu at (259.3, 117.2)
- added R42: 20, Resistor_SMD:R_0805_2012Metric, F.Cu at (256.0, 127.2)
- added R43: 20, Resistor_SMD:R_0805_2012Metric, B.Cu at (250.8, 116.9)
- added R44: 20, Resistor_SMD:R_0805_2012Metric, B.Cu at (254.7, 117.7)
- D39, D40, D41: footprint Diode_SMD:D_SOD-123 -> Diode_SMD:D_SOD-323
Connections:
- U2 pad 3: /LCD1_CS -> Net-(U2-Pad3)
- U2 pad 4: /LCD1_RST -> Net-(U2-Pad4)
- U2 pad 5: /LCD1_DC -> Net-(U2-Pad5)
- U2 pad 6: /MOSI -> Net-(U2-Pad6)
- U2 pad 7: /SCK -> Net-(U2-Pad7)
Routing:
- net +3.3V: track 228.5 -> 257.4 mm, vias 8 -> 10
- net GND: track 314.6 -> 327.0 mm, vias 3 -> 5
- net /LCD1_CS: track 46.2 -> 35.3 mm, vias 1 -> 2
- net Net-(U2-Pad3): track 0.00 -> 9.28 mm, vias 0 -> 1
- net /MOSI: track 78.6 -> 70.1 mm, vias 2 -> 3
- net Net-(U2-Pad6): track 0.00 -> 7.27 mm, vias 0 -> 1
- net /LCD1_DC: track 50.9 -> 43.8 mm, vias 1 -> 2
- net Net-(U2-Pad4): track 0.00 -> 6.52 mm, vias 0 -> 1
- net Net-(U2-Pad5): track 0.00 -> 6.27 mm, vias 0 -> 1
- net unconnected-(U3-Pad40): track 0.00 -> 5.99 mm, vias 0 -> 1
- net unconnected-(U3-Pad43): track 0.00 -> 5.61 mm, vias 0 -> 1
- net /LCD1_RST: track 58.3 -> 52.9 mm, vias 1 -> 2
- net /SCK: track 86.8 -> 81.8 mm
- net unconnected-(U3-Pad39): track 0.00 -> 4.72 mm, vias 0 -> 1
- net unconnected-(U3-Pad42): track 0.00 -> 4.46 mm, vias 0 -> 1
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- added copper zone on B.Cu, net Net-(C4-Pad1)
- removed copper zone on B.Cu, net +3.3V
Other:
- board text removed: "ALL VIA INTERAL DIAMETERS NEED TO BE >= 5mm (for fly wiring) Also untented"
- board text removed: "Mounting holes are cutting into traces, we need to consider creating more board for these holes also consider the screw head that will rest on top of the hole"
- board text removed: "Once done routing, for unused pins, draw out traces and attach vias (assign nets in schematic) this will allow fly wiring if we smoke a pin"
- board text removed: "The switches unfortunately need to be re-spaced. They are 19mm apart from center to center, we need the horizontal distance to be 19mm, center to center distance will be greater than 19mm because of trig & stuff"
- board text removed: "USB receptacles should be spaced a little farther apart to account for usb cable housing clearance (cables may hit each other)"
