File: Splitboard-A/Splitboard-A.kicad_sch (KiCad schematic)
At the start: 125 parts, among them J1 USB_C_Receptacle_USB2.0, J2 USB_C_Receptacle, J3 Conn_01x06, K1 KEYSW, K10 KEYSW, K11 KEYSW, K12 KEYSW, K13 KEYSW, K14 KEYSW, K15 KEYSW, K16 KEYSW, K17 KEYSW, K18 KEYSW, K19 KEYSW, K2 KEYSW, K20 KEYSW, K21 KEYSW, K22 KEYSW, K23 KEYSW, K24 KEYSW, K25 KEYSW, K26 KEYSW, K27 KEYSW, K28 KEYSW, K29 KEYSW, K3 KEYSW, K30 KEYSW, K31 KEYSW, K32 KEYSW, K33 KEYSW, K34 KEYSW, K35 KEYSW, K36 KEYSW, K37 KEYSW, K38 KEYSW, K4 KEYSW, K5 KEYSW, K6 KEYSW, K7 KEYSW, K8 KEYSW, K9 KEYSW, SW1 RotaryEncoder, SW2 SW_Push, U1 SIT2024BA-S2-33E-8.000000G, U2 CR2013-MI2120, U3 STM32F407VGTx, U4 AMS1117-3.3, U5 USBUF02W6

Commit message: Splitboard B schematic completed, added some additional notes on board A
Parts:
- SW1: footprint Rotary_Encoder:RotaryEncoder_Alps_EC12E_Vertical_H20mm -> Rotary_Encoder:RotaryEncoder_Alps_EC11E-Switch_Vertical_H20mm
Other:
- note added: "10K pullup resistors in case internal don't work These may also end up being 1k"
- note added: "There is an embedded pull up on D+ (for device speed selection)"
- note removed: "10K pullup resistors in case internal don't work"
Changed lines of the file:
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@@
     (effects (font (size 1.27 1.27)) (justify left bottom))
   )
+  (text "There is an embedded pull up on D+\n(for device speed selection)"
+    (at 78.3336 67.3608 0)
+    (effects (font (size 1.27 1.27)) (justify left bottom))
+  )
   (text "Need to make sure this is all symmetrical" (at 106.68 182.88 0)
     (effects (font (size 1.27 1.27)) (justify left bottom))
@@
     (effects (font (size 1.27 1.27)) (justify left bottom))
   )
-  (text "10K pullup resistors\nin case internal don't work" (at 196.85 223.52 0)
+  (text "10K pullup resistors\nin case internal don't work\nThese may also end up being 1k"
+    (at 191.008 224.3328 0)
     (effects (font (size 1.27 1.27)) (justify left bottom))
   )
@@
       (effects (font (size 1.27 1.27)) (justify left))
     )
-    (property "Footprint" "Rotary_Encoder:RotaryEncoder_Alps_EC12E_Vertical_H20mm" (id 2) (at 226.06 354.076 0)
+    (property "Footprint" "Rotary_Encoder:RotaryEncoder_Alps_EC11E-Switch_Vertical_H20mm" (id 2) (at 226.06 354.076 0)
       (effects (font (size 1.27 1.27)) hide)
     )
@@
     )
     (path "/38fe4bc3-8fec-480e-9eda-33bcbef5df4c"
-      (reference "SW1") (unit 1) (value "RotaryEncoder") (footprint "Rotary_Encoder:RotaryEncoder_Alps_EC12E_Vertical_H20mm")
+      (reference "SW1") (unit 1) (value "RotaryEncoder") (footprint "Rotary_Encoder:RotaryEncoder_Alps_EC11E-Switch_Vertical_H20mm")
     )
     (path "/aae1d1b8-ecea-4dc3-9e3b-62424a309ff4"

Commit message: Splitboard A schematic completed (added mosi and sck)
Connections:
- net LCD2_RESET is gone; now on net LCD2_RST: U3.68 (PA9)
- net MOSI: now also U3.18 (PC3)
- net SCK: now also U3.52 (PB13)
- net LCD1_RESET renamed LCD1_RST
Changed lines of the file:
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@@
+    (stroke (width 0) (type default) (color 0 0 0 0))
+  )
+  (wire (pts (xy 299.72 217.17) (xy 294.64 217.17))
     (stroke (width 0) (type default) (color 0 0 0 0))
   )
@@
   )
   (wire (pts (xy 82.55 144.78) (xy 82.55 147.32))
+    (stroke (width 0) (type default) (color 0 0 0 0))
+  )
+  (wire (pts (xy 299.72 199.39) (xy 294.64 199.39))
     (stroke (width 0) (type default) (color 0 0 0 0))
   )
@@
     (effects (font (size 1.27 1.27)) (justify left bottom))
   )
+  (label "SCK" (at 299.72 199.39 0)
+    (effects (font (size 1.27 1.27)) (justify left bottom))
+  )
   (label "RCC_OSC_IN" (at 234.95 158.75 0)
     (effects (font (size 1.27 1.27)) (justify left bottom))
@@
     (effects (font (size 1.27 1.27)) (justify left bottom))
   )
-  (label "LCD2_RESET" (at 299.72 146.05 0)
+  (label "LCD2_RST" (at 299.72 146.05 0)
     (effects (font (size 1.27 1.27)) (justify left bottom))
   )
@@
     (effects (font (size 1.27 1.27)) (justify left bottom))
   )
-  (label "LCD1_RESET" (at 450.85 73.66 0)
+  (label "LCD1_RST" (at 450.85 73.66 0)
     (effects (font (size 1.27 1.27)) (justify left bottom))
   )
@@
   )
   (label "row6" (at 245.11 224.79 0)
+    (effects (font (size 1.27 1.27)) (justify left bottom))
+  )
+  (label "MOSI" (at 299.72 217.17 0)
     (effects (font (size 1.27 1.27)) (justify left bottom))
   )
@@
     (effects (font (size 1.27 1.27)) (justify left bottom))
   )
-  (label "LCD1_RESET" (at 299.72 148.59 0)
-    (effects (font (size 1.27 1.27)) (justify left bottom))
-  )
+  (label "LCD1_RST" (at 299.72 148.59 0)
+    (effects (font (size 1.27 1.27)) (justify left bottom))
+  )
