File: Splitboard-B/_autosave-Splitboard-B.kicad_sch (KiCad schematic)
At the start: 109 parts, among them J4 USB_C_Receptacle, K39 KEYSW, K40 KEYSW, K41 KEYSW, K42 KEYSW, K43 KEYSW, K44 KEYSW, K45 KEYSW, K46 KEYSW, K47 KEYSW, K48 KEYSW, K49 KEYSW, K50 KEYSW, K51 KEYSW, K52 KEYSW, K53 KEYSW, K54 KEYSW, K55 KEYSW, K56 KEYSW, K57 KEYSW, K58 KEYSW, K59 KEYSW, K60 KEYSW, K61 KEYSW, K62 KEYSW, K63 KEYSW, K64 KEYSW, K65 KEYSW, K66 KEYSW, K67 KEYSW, K68 KEYSW, K69 KEYSW, K70 KEYSW, K71 KEYSW, K72 KEYSW, K73 KEYSW, K74 KEYSW, K75 KEYSW, K76 KEYSW, U5 CR2013-MI2120

Commit message: Added Joe's suggestions & notes to schematic & pcb
Parts:
- R6, R8: value 4.7K -> 4K7
Changed lines of the file:
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@@
       (effects (font (size 1.27 1.27)) (justify left))
     )
-    (property "Value" "4.7K" (id 1) (at 238.76 248.92 0)
+    (property "Value" "4K7" (id 1) (at 238.76 248.92 0)
       (effects (font (size 1.27 1.27)) (justify left))
     )
@@
       (effects (font (size 1.27 1.27)) (justify left))
     )
-    (property "Value" "4.7K" (id 1) (at 231.14 248.92 0)
+    (property "Value" "4K7" (id 1) (at 231.14 248.92 0)
       (effects (font (size 1.27 1.27)) (justify left))
     )
@@
     )
     (path "/d2a3d573-3fdc-446c-83c0-323323c0f869"
-      (reference "R6") (unit 1) (value "4.7K") (footprint "")
+      (reference "R6") (unit 1) (value "4K7") (footprint "")
     )
     (path "/cf07b8d4-ac6a-4205-956c-af4a10ed30b8"
-      (reference "R8") (unit 1) (value "4.7K") (footprint "")
+      (reference "R8") (unit 1) (value "4K7") (footprint "")
     )
     (path "/ac921aa6-3e71-4671-9a11-bd089ae29fe6"
