File: Splitboard-B/Splitboard-B.kicad_pcb (KiCad board)
At the start: 2 copper layers, 185 x 161.7 mm, 133 parts, among them J1 USB_C_Receptacle, J2 Conn_01x09, K1 KEYSW, K10 KEYSW, K11 KEYSW, K12 KEYSW, K13 KEYSW, K14 KEYSW, K15 KEYSW, K16 KEYSW, K17 KEYSW, K18 KEYSW, K19 KEYSW, K2 KEYSW, K20 KEYSW, K21 KEYSW, K22 KEYSW, K23 KEYSW, K24 KEYSW, K25 KEYSW, K26 KEYSW, K27 KEYSW, K28 KEYSW, K29 KEYSW, K3 KEYSW, K30 KEYSW, K31 KEYSW, K32 KEYSW, K33 KEYSW, K34 KEYSW, K35 KEYSW, K36 KEYSW, K37 KEYSW, K38 KEYSW, K4 KEYSW, K5 KEYSW, K6 KEYSW, K7 KEYSW, K8 KEYSW, K9 KEYSW, SW1 RotaryEncoder, U1 CR2013-MI2120, U2 MCP23017_SP, U3 AMS1117-3.3

Commit message: Layout changes
Parts:
- D39: footprint Diode_SMD:D_SOD-123 -> Diode_SMD:D_SOD-323
- J2: moved to B.Cu
- moved J2 20.8 mm to (59.0, 73.7)
- moved R6 10.3 mm to (60.9, 149.4)
- moved C1 10.3 mm to (83.9, 140.6)
- moved R3 10.3 mm to (83.9, 145.8)
- moved R8 10.3 mm to (84.0, 137.2)
- moved R9 10.3 mm to (54.6, 138.4)
- moved C2 10.3 mm to (53.7, 141.7)
- moved C3 10.3 mm to (57.0, 145.4)
- moved R10 10.3 mm to (57.0, 148.0)
- moved R4 10.3 mm to (60.7, 136.7)
- moved R5 10.3 mm to (60.7, 140.7)
- moved R7 10.3 mm to (61.2, 145.7)
- moved SW1 10.3 mm to (65.7, 140.7)
- moved C7 0.25 mm to (72.7, 62.0)
Routing:
- net +3.3V: track 249.6 -> 286.0 mm, vias 5 -> 7
- net Net-(R9-Pad2): track 103.1 -> 123.6 mm
- net /LCD2_RST: track 60.2 -> 73.1 mm
- net /SDA: track 114.8 -> 103.6 mm, vias 3 -> 4
- net Net-(R10-Pad2): track 95.8 -> 106.9 mm
- net /LCD2_DC: track 56.0 -> 66.6 mm
- net /col5: track 130.3 -> 140.8 mm
- net /MOSI: track 62.1 -> 71.3 mm
- net VBUS: track 135.6 -> 128.9 mm
- net /SCK: track 65.4 -> 71.2 mm, vias 0 -> 1
- net /SCL: track 127.8 -> 123.0 mm
- net Net-(R22-Pad1): track 14.0 -> 18.1 mm
- net Net-(R8-Pad2): track 64.6 -> 60.7 mm
- net Net-(J1-PadA10): track 61.9 -> 65.2 mm
- net Net-(J1-PadA11): track 56.0 -> 58.7 mm
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Other:
- board text added: "1"
- board text added: "Split Keyboard Side B ECE 477 Group 4 Fall 2022 Senior Design Andrew Smolensky Logan Stapleton Joe Zobel Justin Selbo"

Commit message: Addes rseries for LCD and added extra vias
Routing:
- net Net-(D39-Pad1): track 0.00 -> 2.79 mm
- net /col3: track 185.1 -> 185.9 mm
- net /col1: track 196.1 -> 196.8 mm
Other:
- board text removed: "ALL VIA INTERAL DIAMETERS NEED TO BE >= 5mm (for fly wiring) Also untented"
- board text removed: "The switches unfortunately need to be re-spaced. They are 19mm apart from center to center, we need the horizontal distance to be 19mm, center to center distance will be greater than 19mm because of trig & stuff"
- board text removed: "we need to consider creating more board for these holes consider the screw head that will rest on top of the hole"
